File: optiga-tpm-module.kicad_pcb (KiCad board)
At the start: 2 copper layers, 20 x 29 mm, 40 parts, among them J1 Plug_Samtec_ERM5_2x20_ERM5-02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, U1 SLB9672XU20FW1624XTMA1

Commit message: [#104798] Clean up the schematic, add termal vias to IC
Parts:
- added TP1: TP_0.75mm_SMD, antmicro-footprints:TP_SMD_0.75mm, F.Cu at (0.50, 0.50)
Routing:
- net GND: vias 8 -> 13

Commit message: [#104798] pcb: import TP1 from schematic, remove duplicate
Parts:
- removed the TP1 at (338.9, 234.6)
- moved TP1 411.4 mm to (338.9, 234.6)
Changed lines of the file:
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@@
 		(capping no)
 		(filling no)
-		(zone_defaults)
 		(pcbplotparams
 			(layerselection 0x00000000_00000000_55555555_5755f5ff)
@@
 	(footprint "antmicro-footprints:TP_SMD_0.75mm"
 		(layer "F.Cu")
-		(at 0.5 0.5)
-		(property "Reference" "TP1"
-			(at 0 -0.6 0)
-			(layer "F.SilkS")
-			(effects
-				(font
-					(size 0.7 0.7)
-					(thickness 0.15)
-				)
-				(justify left bottom)
-			)
-		)
-		(property "Value" "TP_0.75mm_SMD"
-			(at 0 1.2 0)
-			(layer "F.Fab")
-			(effects
-				(font
-					(size 0.7 0.7)
-					(thickness 0.15)
-				)
-				(justify left bottom)
-			)
-		)
-		(property "Datasheet" ""
-			(at 0 0 0)
-			(layer "F.Fab")
-			(hide yes)
-			(effects
-				(font
-					(size 1.27 1.27)
-					(thickness 0.15)
-				)
-			)
-		)
-		(property "Description" "SMT test point"
-			(at 0 0 0)
-			(layer "F.Fab")
-			(hide yes)
-			(effects
-				(font
-					(size 1.27 1.27)
-					(thickness 0.15)
-				)
-			)
-		)
-		(property "MPN" ""
-			(at 0 0 0)
-			(unlocked yes)
-			(layer "F.Fab")
-			(hide yes)
-			(effects
-				(font
-					(size 1 1)
-					(thickness 0.15)
-				)
-			)
-		)
-		(property "Manufacturer" ""
-			(at 0 0 0)
-			(unlocked yes)
-			(layer "F.Fab")
-			(hide yes)
-			(effects
-				(font
-					(size 1 1)
-					(thickness 0.15)
-				)
-			)
-		)
-		(property "Author" "Antmicro"
-			(at 0 0 0)
-			(unlocked yes)
-			(layer "F.Fab")
-			(hide yes)
-			(effects
-				(font
-					(size 1 1)
-					(thickness 0.15)
-				)
-			)
-		)
-		(property "License" "Apache-2.0"
-			(at 0 0 0)
-			(unlocked yes)
-			(layer "F.Fab")
-			(hide yes)
-			(effects
-				(font
-					(size 1 1)
-					(thickness 0.15)
-				)
-			)
-		)
-		(sheetname "/")
-		(sheetfile "optiga-tpm-module.kicad_sch")
-		(units
-			(unit
-				(name "A")
-				(pins "1")
-			)
-		)
-		(attr exclude_from_bom)
-		(stackup
-			(layer "F.Cu")
-			(layer "B.Cu")
-			(layer "User.1")
-			(layer "User.2")
-			(layer "User.3")
-			(layer "User.4")
-			(layer "User.5")
-			(layer "User.6")
-			(layer "User.7")
-			(layer "User.8")
-			(layer "User.9")
-		)
-		(duplicate_pad_numbers_are_jumpers no)
-		(fp_circle
-			(center 0 0)
-			(end 0.475 0)
-			(stroke
-				(width 0.05)
-				(type default)
-			)
-			(fill no)
-			(layer "F.CrtYd")
-		)
-		(fp_text user "${REFERENCE}"
-			(at -0.4 2.7 0)
-			(layer "F.Fab")
-			(effects
-				(font
-					(size 0.7 0.7)
-					(thickness 0.15)
-				)
-				(justify left bottom)
-			)
-		)
-		(fp_text user "Author: Antmicro"
-			(at -0.4 3.901 0)
-			(layer "F.Fab")
-			(effects
-				(font
-					(size 0.7 0.7)
-					(thickness 0.15)
-				)
-				(justify left bottom)
-			)
-		)
-		(fp_text user "License: Apache-2.0"
-			(at -0.4 5.101 0)
-			(layer "F.Fab")
-			(effects
-				(font
-					(size 0.7 0.7)
-					(thickness 0.15)
-				)
-				(justify left bottom)
-			)
-		)
-		(pad "1" smd circle
-			(at 0 0)
-			(size 0.75 0.75)
-			(layers "F.Cu" "F.Mask")
-			(net "GND")
-			(pinfunction "1_1")
-			(pintype "passive")
-		)
-		(embedded_fonts no)
-	)
-	(footprint "antmicro-footprints:TP_SMD_0.75mm"
-		(layer "F.Cu")
-		(at 338.9 234.55)
+		(at 338.85 234.55)
 		(property "Reference" "TP1"
 			(at 0 -0.6 0)
@@
 	)
 	(segment
+		(start 341.08 235.7)
+		(end 342.25 235.7)
+		(width 0.3)
+		(layer "F.Cu")
+		(net "Net-(D1-A)")
+	)
+	(segment
 		(start 341.879 226.95)
 		(end 341.009 226.95)
@@
 	)
 	(segment
-		(start 341.08 235.7)
-		(end 342.25 235.7)
-		(width 0.3)
-		(layer "F.Cu")
-		(net "Net-(D1-A)")
-	)
-	(segment
